File: orblink.brd (EAGLE design)
At the start: 27 x 27 mm, 13 parts, among them U1 ATTINY

Commit message: Switched LED and USB pin
Parts:
- R1: value 68 -> 220
- R2: value 68 -> 330
- R3: value 68 -> 150
Connections:
- net GRN: now also U1.5; no longer U1.2
- net N$4: now also U1.2; no longer U1.5
Routing:
- net N$4: track 4.37 -> 13.9 mm
- net GRN: track 15.0 -> 19.8 mm
Other:
- board text added: "OrBlink"
- board text added: "v2.0"
Changed lines of the file:
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@@
 <setting verticaltext="up"/>
 </settings>
-<grid distance="20" unitdist="mil" unit="mil" style="lines" multiple="1" display="yes" altdistance="0.005" altunitdist="inch" altunit="inch"/>
+<grid distance="10" unitdist="mil" unit="mil" style="lines" multiple="1" display="yes" altdistance="0.005" altunitdist="inch" altunit="inch"/>
 <layers>
 <layer number="1" name="Top" color="4" fill="1" visible="yes" active="yes"/>
@@
 <text x="8.25" y="21.25" size="0.762" layer="25" font="vector" ratio="14">VCC</text>
 <text x="12.954" y="14.986" size="0.6604" layer="25" font="vector" ratio="12">LED</text>
+<text x="11.684" y="25.4" size="0.8128" layer="21" font="vector">v2.0</text>
+<text x="9.652" y="17.272" size="1.4224" layer="21" font="vector">OrBlink</text>
 </plain>
 <attributes>
@@
 <attribute name="NAME" x="9.008" y="20.254" size="0.6604" layer="25" font="vector" ratio="12" rot="R180"/>
 </element>
-<element name="R2" library="SparkFun-Resistors" package="1/6W-RES" value="68" x="6" y="14" smashed="yes" rot="R90">
+<element name="R2" library="SparkFun-Resistors" package="1/6W-RES" value="330" x="6" y="14" smashed="yes" rot="R90">
 <attribute name="NAME" x="6.3148" y="13.4958" size="0.6604" layer="25" font="vector" ratio="12" rot="R90"/>
 </element>
-<element name="R1" library="SparkFun-Resistors" package="1/6W-RES" value="68" x="3.5" y="13.5" smashed="yes" rot="R90">
+<element name="R1" library="SparkFun-Resistors" package="1/6W-RES" value="220" x="3.5" y="13.5" smashed="yes" rot="R90">
 <attribute name="NAME" x="3.8148" y="12.9958" size="0.6604" layer="25" font="vector" ratio="12" rot="R90"/>
 </element>
-<element name="R3" library="SparkFun-Resistors" package="1/6W-RES" value="68" x="8.5" y="14.5" smashed="yes" rot="R90">
+<element name="R3" library="SparkFun-Resistors" package="1/6W-RES" value="150" x="8.5" y="14.5" smashed="yes" rot="R90">
 <attribute name="NAME" x="8.8148" y="13.9958" size="0.6604" layer="25" font="vector" ratio="12" rot="R90"/>
 </element>
@@
 <wire x1="12.22" y1="9.934" x2="12.22" y2="9.89" width="0.4064" layer="1"/>
 </signal>
-<signal name="N$4">
-<contactref element="U1" pad="5"/>
-<contactref element="R5" pad="2"/>
-<wire x1="21" y1="11.5" x2="19.39" y2="9.89" width="0.4064" layer="1"/>
-<wire x1="19.39" y1="9.89" x2="17.3" y2="9.89" width="0.4064" layer="1"/>
-</signal>
 <signal name="D-">
 <contactref element="R5" pad="1"/>
@@
 </signal>
 <signal name="GRN">
-<contactref element="U1" pad="2"/>
 <contactref element="R1" pad="1"/>
 <wire x1="3.5" y1="11" x2="3.5" y2="8.819" width="0.4064" layer="1"/>
 <wire x1="3.5" y1="8.819" x2="6.35" y2="5.969" width="0.4064" layer="1"/>
-<wire x1="6.35" y1="5.969" x2="10.922" y2="5.969" width="0.4064" layer="1"/>
-<wire x1="10.922" y1="5.969" x2="12.22" y2="4.671" width="0.4064" layer="1"/>
-<wire x1="12.22" y1="4.671" x2="12.22" y2="2.27" width="0.4064" layer="1"/>
+<wire x1="6.35" y1="5.969" x2="15.113" y2="5.969" width="0.4064" layer="1"/>
+<contactref element="U1" pad="5"/>
+<wire x1="15.113" y1="5.969" x2="17.272" y2="8.128" width="0.4064" layer="1"/>
+<wire x1="17.272" y1="8.128" x2="17.272" y2="9.862" width="0.4064" layer="1"/>
+<wire x1="17.272" y1="9.862" x2="17.3" y2="9.89" width="0.4064" layer="1"/>
 </signal>
 <signal name="BLU">
 <contactref element="U1" pad="3"/>
 <contactref element="R2" pad="1"/>
-<wire x1="6" y1="11.5" x2="6" y2="8.097" width="0.4064" layer="1"/>
-<wire x1="6" y1="8.097" x2="7.366" y2="6.731" width="0.4064" layer="1"/>
-<wire x1="7.366" y1="6.731" x2="12.7" y2="6.731" width="0.4064" layer="1"/>
-<wire x1="12.7" y1="6.731" x2="14.76" y2="4.671" width="0.4064" layer="1"/>
-<wire x1="14.76" y1="4.671" x2="14.76" y2="2.27" width="0.4064" layer="1"/>
+<wire x1="6" y1="11.5" x2="6" y2="8.097" width="0.4064" layer="16"/>
+<wire x1="6" y1="8.097" x2="7.366" y2="6.731" width="0.4064" layer="16"/>
+<wire x1="7.366" y1="6.731" x2="12.7" y2="6.731" width="0.4064" layer="16"/>
+<wire x1="12.7" y1="6.731" x2="14.76" y2="4.671" width="0.4064" layer="16"/>
+<wire x1="14.76" y1="4.671" x2="14.76" y2="2.27" width="0.4064" layer="16"/>
 </signal>
 <signal name="N$1">
@@
 <wire x1="15.405" y1="15.71" x2="15.405" y2="13.5" width="0.4064" layer="1"/>
 </signal>
+<signal name="N$4">
+<contactref element="U1" pad="2"/>
+<contactref element="R5" pad="2"/>
+<wire x1="12.22" y1="2.27" x2="14.522" y2="4.572" width="0.4064" layer="1"/>
+<wire x1="14.522" y1="4.572" x2="16.256" y2="4.572" width="0.4064" layer="1"/>
+<wire x1="16.256" y1="4.572" x2="21" y2="9.316" width="0.4064" layer="1"/>
+<wire x1="21" y1="9.316" x2="21" y2="11.5" width="0.4064" layer="1"/>
+</signal>
 </signals>
